File: P3-FourChannelRelayModule/nodemcurelay.brd (EAGLE design)
At the start: 60 x 80 mm, 22 parts, among them IC1 7812T, K1 CQ1-12V, K2 CQ1-12V, K3 CQ1-12V, K4 CQ1-12V, T1 2N2222, T2 2N2222, T3 2N2222, T4 2N2222

Commit message: Updated Relay Boards
Parts:
- added X1, X2, X3, X4: (no value), con-ptr500:AK300/3
Connections:
- new net N$11: K1.NC, X1.1
- new net N$17: K1.C, X1.2
- new net N$18: K2.NC, X2.1
- new net N$19: K2.C, X2.2
- new net N$20: K2.NO, X2.3
- new net N$21: K3.NO, X3.3
- new net N$22: K3.NC, X3.1
- new net N$23: K3.C, X3.2
- new net N$24: K4.NO, X4.3
- new net N$25: K4.C, X4.2
- new net N$26: K4.NC, X4.1
- new net N$7: K1.NO, X1.3
Routing:
- net N$25: track 0.00 -> 24.3 mm
- net N$17: track 0.00 -> 24.1 mm
- net N$23: track 0.00 -> 23.6 mm
- net N$19: track 0.00 -> 23.6 mm
- net 12V: track 156.9 -> 176.1 mm
- net N$26: track 0.00 -> 11.6 mm
- net N$24: track 0.00 -> 11.6 mm
- net N$7: track 0.00 -> 11.4 mm
- net N$11: track 0.00 -> 11.4 mm
- net N$22: track 0.00 -> 10.9 mm
- net N$21: track 0.00 -> 10.9 mm
- net N$20: track 0.00 -> 10.9 mm
- net N$18: track 0.00 -> 10.9 mm
- net N$5: track 9.17 -> 10.2 mm
Other:
- board size 60 x 80 mm -> 73 x 80 mm
